Commit message: complete 6DOF robot arm urdf with testing joints motions

File: src/learn_robotics_with_ROS_youtube_channel/robot_arm/urdf/robot_arm.urdf.xacro (robot description, xacro)
@@ -3,64 +3,166 @@
 <robot name="robot_arm" xmlns:xacro="http://ros.org/wiki/xacro">
   <xacro:include filename="robot_arm_macros.xacro"/>
+  <xacro:include filename="gripper.xacro"/>
+  <!-- ====== WORLD LINK ====== -->
   <link name="world"/>
-  <joint name="world_base_link" type="fixed">
-    <parent link="world"/>
-    <child link="base_link"/>
-    <origin xyz="0 0 0" rpy="0 0 0"/>
-  </joint>
-  <!-- Links using macros and mass param -->
-  <xacro:link_cylinder name="base_link" xyz="0 0 0.025" rpy="0 0 0" radius="0.1" length="0.05" mass="1.0"/>
-  <xacro:link_cylinder name="link1" xyz="0 0 0.132" rpy="0 0 0" radius="0.05" length="0.264" mass="0.6"/>
-  <xacro:link_cylinder name="link2" xyz="0 0 0.425" rpy="0 0 0" radius="0.05" length="0.850" mass="0.7"/>
-  <!-- <xacro:link_cylinder name="link3" xyz="0 0 0.340" rpy="0 0 0" radius="0.05" length="0.680" mass="0.8"/>
-  <xacro:link_cylinder name="link4" xyz="0 0 0.065" rpy="0 0 0" radius="0.05" length="0.130" mass="0.5"/>
-  <xacro:link_cylinder name="link5" xyz="0 0 0" rpy="0 0 0" radius="0.05" length="0.170" mass="0.3"/>
-  <xacro:link_box name="gripper_base" xyz="0 0 0.0125" rpy="0 0 0" w="0.03" h="0.15" d="0.03" mass="0.2"/>
-  <xacro:link_box name="gripper_right" xyz="0 0 0.05" rpy="0 0 0" w="0.01" h="0.01" d="0.10" mass="0.05"/>
-  <xacro:link_box name="gripper_left" xyz="0 0 0.05" rpy="0 0 0" w="0.01" h="0.01" d="0.10" mass="0.05"/> -->
-    <!-- For every controlled joint -->
-    <!-- <xacro:transmission_effort name="trans_base_link_link1" joint_name="base_link_link1" actuator_name="motor_base_link_link1"/>
-    <xacro:transmission_effort name="trans_link1_link2" joint_name="link1_link2" actuator_name="motor_link1_link2"/>
-    <xacro:transmission_effort name="trans_link2_link3" joint_name="link2_link3" actuator_name="motor_link2_link3"/>
-    <xacro:transmission_effort name="trans_link3_link4" joint_name="link3_link4" actuator_name="motor_link3_link4"/>
-    <xacro:transmission_effort name="trans_link4_link5" joint_name="link4_link5" actuator_name="motor_link4_link5"/>
-    <xacro:transmission_effort name="trans_link5_gripper_base" joint_name="link5_gripper_base" actuator_name="motor_link5_gripper_base"/> -->
-    <!-- For the gripper -->
-    <!-- <xacro:transmission_effort name="trans_gripper_base_gripper_right" joint_name="gripper_base_gripper_right" actuator_name="motor_gripper_base_gripper_right"/>
-    <xacro:transmission_effort name="trans_gripper_base_gripper_left" joint_name="gripper_base_gripper_left" actuator_name="motor_gripper_base_gripper_left"/> -->
-  <!-- Joints using macros -->
-  <xacro:joint name="base_link_link1" type="revolute" parent="base_link" child="link1" axis="0 0 1"
-      lower="-3.14159" upper="3.14159" velocity="0.5" effort="1000.0"
-      xyz="0 0 0.05" rpy="0 0 0"/>
-  <xacro:joint name="link1_link2" type="revolute" parent="link1" child="link2" axis="1 0 0"
-      lower="-2.5" upper="2.5" velocity="0.5" effort="1000.0"
-      xyz="0.1 0 0.264" rpy="0 0 0"/>
-  <!-- <xacro:joint name="link2_link3" type="revolute" parent="link2" child="link3" axis="1 0 0"
-      lower="-3.14" upper="3.14" velocity="0.5" effort="1000.0"
-      xyz="-0.1 0 0.850" rpy="0 0 0"/>
-  <xacro:joint name="link3_link4" type="revolute" parent="link3" child="link4" axis="1 0 0"
-      lower="-3.14" upper="3.14" velocity="0.5" effort="1000.0"
-      xyz="0.1 0.0 0.680" rpy="0.0 0.0 0.0"/>
-  <xacro:joint name="link4_link5" type="revolute" parent="link4" child="link5" axis="0 1 0"
-      lower="-3.14" upper="3.14" velocity="0.5" effort="1000.0"
-      xyz="0 0 0.180" rpy="1.570 0.0 0.0"/>
-  <xacro:joint name="link5_gripper_base" type="revolute" parent="link5" child="gripper_base" axis="0 0 1"
-      lower="-3.14" upper="3.14" velocity="0.5" effort="1000.0"
-      xyz="0 0 0.085" rpy="0 0 1.57"/>
-  <xacro:joint name="gripper_base_gripper_right" type="prismatic" parent="gripper_base" child="gripper_right" axis="0 1 0"
-      lower="0.0" upper="0.055" velocity="0.5" effort="1000.0"
-      xyz="0 -0.065 0.03" rpy="0 0 0"/>
-  <xacro:joint name="gripper_base_gripper_left" type="prismatic" parent="gripper_base" child="gripper_left" axis="0 -1 0"
-      lower="0.0" upper="0.055" velocity="0.5" effort="1000.0"
-      xyz="0 0.065 0.03" rpy="0 0 0"/> -->
-  <!-- Modern ros2_control block (NO <gazebo>!) -->
+  <!-- ====== FIX ROBOT TO WORLD ====== -->
+  <xacro:cobot_joint
+    name="world_base_link"
+    type="fixed"
+    parent="world"
+    child="base_link"
+    axis="0 0 0"
+    limit_l="0"
+    limit_u="0"
+    limit_v="0"
+    limit_e="0"
+    origin_xyz="0 0 0"
+    origin_rpy="0 0 0"/>
+  <!-- ====== ARM LINKS ====== -->
+  <!-- Base link -->
+  <xacro:link_cylinder
+    name="base_link"
+    xyz="0 0 0.025"
+    rpy="0 0 0"
+    radius="0.1"
+    length="0.05"
+    mass="1.0"
+    ixx="0.00270833"
+    iyy="0.00270833"
+    izz="0.005"/>
+  <!-- Link 1 -->
+  <xacro:link_cylinder
+    name="link1"
+    xyz="0 0 0.132"
+    rpy="0 0 0"
+    radius="0.05"
+    length="0.264"
+    mass="0.6"
+    ixx="0.005808"
+    iyy="0.005808"
+    izz="0.00075"/>
+  <!-- Link 2 -->
+  <xacro:link_cylinder
+    name="link2"
+    xyz="0 0 0.425"
+    rpy="0 0 0"
+    radius="0.05"
+    length="0.850"
+    mass="0.7"
+    ixx="0.042583"
+    iyy="0.042583"
+    izz="0.000875"/>
+  <!-- Link 3 (commented - uncomment when ready) -->
+  <xacro:link_cylinder
+    name="link3"
+    xyz="0 0 0.340"
+    rpy="0 0 0"
+    radius="0.05"
+    length="0.680"
+    mass="0.8"
+    ixx="0.038293"
+    iyy="0.038293"
+    izz="0.001"/>
+  <!-- Link 4 (commented - uncomment when ready) -->
+  <xacro:link_cylinder
+    name="link4"
+    xyz="0 0 0.065"
+    rpy="0 0 0"
+    radius="0.05"
+    length="0.130"
+    mass="0.5"
+    ixx="0.003646"
+    iyy="0.003646"
+    izz="0.000625"/>
+  <!-- Link 5 (commented - uncomment when ready) -->
+  <xacro:link_cylinder
+    name="link5"
+    xyz="0 0 0.035"
+    rpy="0 0 0"
+    radius="0.05"
+    length="0.170"
+    mass="0.3"
+    ixx="0.00225"
+    iyy="0.00225"
+    izz="0.000375"/>
+  <!-- Gripper (commented - uncomment when ready with link5) -->
+  <xacro:gripper_connector_link/>
+  <xacro:gripper_right_finger_link/>
+  <xacro:gripper_left_finger_link/>
+  <!-- ====== ARM JOINTS ====== -->
+  <!-- Joint: base_link to link1 -->
+  <xacro:cobot_joint
+    name="base_link_link1"
+    type="revolute"
+    parent="base_link"
+    child="link1"
+    axis="0 0 1"
+    limit_l="-3.14159"
+    limit_u="3.14159"
+    limit_v="0.5"
+    limit_e="1000.0"
+    origin_xyz="0 0 0.05"
+    origin_rpy="0 0 0"/>
+  <!-- Joint: link1 to link2 -->
+  <xacro:cobot_joint
+    name="link1_link2"
+    type="revolute"
+    parent="link1"
+    child="link2"
+    axis="1 0 0"
+    limit_l="-2.5"
+    limit_u="2.5"
+    limit_v="0.5"
+    limit_e="1000.0"
+    origin_xyz="0.1 0 0.264"
+    origin_rpy="0 0 0"/>
+  <!-- Joint: link2 to link3 (commented - uncomment when ready) -->
+  <xacro:cobot_joint
+    name="link2_link3"
+    type="revolute"
+    parent="link2"
+    child="link3"
+    axis="1 0 0"
+    limit_l="-3.14"
+    limit_u="3.14"
+    limit_v="0.5"
+    limit_e="1000.0"
+    origin_xyz="-0.1 0 0.850"
+    origin_rpy="0 0 0"/>
+  <!-- Joint: link3 to link4 (commented - uncomment when ready) -->
+  <xacro:cobot_joint
+    name="link3_link4"
+    type="revolute"
+    parent="link3"
+    child="link4"
+    axis="1 0 0"
+    limit_l="-3.14"
+    limit_u="3.14"
+    limit_v="0.5"
+    limit_e="1000.0"
+    origin_xyz="0.1 0 0.680"
+    origin_rpy="0 0 0"/>
+  <!-- Joint: link4 to link5 (commented - uncomment when ready) -->
+  <xacro:cobot_joint
+    name="link4_link5"
+    type="revolute"
+    parent="link4"
+    child="link5"
+    axis="0 1 0"
+    limit_l="-3.14"
+    limit_u="3.14"
+    limit_v="0.5"
+    limit_e="1000.0"
+    origin_xyz="0 0 0.180"
+    origin_rpy="1.57 0 0"/>
+  <xacro:gripper_connector_joint parent="link5" origin_xyz="0 0 0.135"/>
+  <xacro:gripper_right_finger_joint />
+  <xacro:gripper_left_finger_joint />
+  <!-- ====== ROS2_CONTROL CONFIGURATION ====== -->
   <ros2_control name="RobotController" type="system">
     <hardware>
       <plugin>gz_ros2_control/GazeboSimSystem</plugin>
-      <!-- <param name="position_proportional_gain">1.0</param>
-      <param name="position_integral_gain">0.5</param>
-      <param name="position_derivative_gain">1.0</param> -->
     </hardware>
-    <!-- Repeat for all controlled joints -->
+    <!-- Active arm joints -->
     <joint name="base_link_link1">
       <command_interface name="position"/>
@@ -73,34 +175,41 @@
       <state_interface name="velocity"/>
     </joint>
-    <!-- <joint name="link2_link3">
-      <command_interface name="effort"/>
-      <state_interface name="position"/>
+    <!-- Additional joints (uncomment when ready) -->
+    <joint name="link2_link3">
+      <command_interface name="position"/>
+      <state_interface name="position"/>
+      <state_interface name="velocity"/>
     </joint>
     <joint name="link3_link4">
-      <command_interface name="effort"/>
-      <state_interface name="position"/>
+      <command_interface name="position"/>
+      <state_interface name="position"/>
+      <state_interface name="velocity"/>
     </joint>
     <joint name="link4_link5">
-      <command_interface name="effort"/>
-      <state_interface name="position"/>
-    </joint>
-    <joint name="link5_gripper_base">
-      <command_interface name="effort"/>
-      <state_interface name="position"/>
-    </joint>
-    <joint name="gripper_base_gripper_right">
-      <command_interface name="effort"/>
-      <state_interface name="position"/>
-    </joint>
-    <joint name="gripper_base_gripper_left">
-      <command_interface name="effort"/>
-      <state_interface name="position"/>
-    </joint> -->
+      <command_interface name="position"/>
+      <state_interface name="position"/>
+      <state_interface name="velocity"/>
+    </joint>
+    <joint name="gripper_connector_joint">
+      <command_interface name="position"/>
+      <state_interface name="position"/>
+      <state_interface name="velocity"/>
+    </joint>
+    <joint name="gripper_right_joint">
+      <command_interface name="position"/>
+      <state_interface name="position"/>
+      <state_interface name="velocity"/>
+    </joint>
+    <joint name="gripper_left_joint">
+      <command_interface name="position"/>
+      <state_interface name="position"/>
+      <state_interface name="velocity"/>
+    </joint>
   </ros2_control>
-<!-- In your robot_arm.urdf.xacro, add back this block -->
+  <!-- ====== GAZEBO PLUGIN ====== -->
   <gazebo>
     <plugin name="gz_ros2_control::GazeboSimROS2ControlPlugin" filename="libgz_ros2_control-system.so">
       <parameters>$(find robot_arm)/config/controller.yaml</parameters>
-        <controller_manager_name>controller_manager</controller_manager_name>
+      <controller_manager_name>controller_manager</controller_manager_name>
     </plugin>
   </gazebo>

File: src/learn_robotics_with_ROS_youtube_channel/robot_arm/urdf/robot_arm_macros.xacro (robot description, xacro)
@@ -2,7 +2,18 @@
 <!-- robot_arm_macros.xacro -->
 <robot xmlns:xacro="http://ros.org/wiki/xacro">
-  <!-- Macro for cylinder link -->
-  <xacro:macro name="link_cylinder" params="name xyz rpy radius length mass">
+  <!-- ====== CYLINDER LINK MACRO ====== -->
+  <xacro:macro name="link_cylinder" params="name xyz rpy radius length mass ixx iyy izz">
     <link name="${name}">
+      <inertial>
+        <origin xyz="0 0 0" rpy="0 0 0"/>
+        <mass value="${mass}"/>
+        <inertia
+          ixx="${ixx}"
+          ixy="0.0"
+          ixz="0.0"
+          iyy="${iyy}"
+          iyz="0.0"
+          izz="${izz}"/>
+      </inertial>
       <visual>
         <geometry>
@@ -17,71 +28,46 @@
         <origin xyz="${xyz}" rpy="${rpy}"/>
       </collision>
-      <inertial>
-        <mass value="${mass}"/>
-        <origin xyz="${xyz}" rpy="${rpy}"/>
-        <inertia
-        ixx="${(1/12.0)*mass*(3*radius*radius + length*length)}"
-        iyy="${(1/12.0)*mass*(3*radius*radius + length*length)}"
-        izz="${0.5*mass*radius*radius}"
-        ixy="0.0" ixz="0.0" iyz="0.0"/>
-      </inertial>
     </link>
   </xacro:macro>
-  <!-- Macro for box link -->
-  <xacro:macro name="link_box" params="name xyz rpy w h d mass">
+  <!-- ====== BOX LINK MACRO ====== -->
+  <xacro:macro name="cobot_link_box" params="name origin_xyz origin_rpy size mass ixx ixy ixz iyy iyz izz">
     <link name="${name}">
+      <inertial>
+        <origin xyz="0 0 0" rpy="0 0 0"/>
+        <mass value="${mass}"/>
+        <inertia
+          ixx="${ixx}"
+          ixy="${ixy}"
+          ixz="${ixz}"
+          iyy="${iyy}"
+          iyz="${iyz}"
+          izz="${izz}"/>
+      </inertial>
       <visual>
         <geometry>
-          <box size="${w} ${h} ${d}"/>
+          <box size="${size}"/>
         </geometry>
-        <origin xyz="${xyz}" rpy="${rpy}"/>
+        <origin xyz="${origin_xyz}" rpy="${origin_rpy}"/>
       </visual>
       <collision>
         <geometry>
-          <box size="${w} ${h} ${d}"/>
+          <box size="${size}"/>
         </geometry>
-        <origin xyz="${xyz}" rpy="${rpy}"/>
+        <origin xyz="${origin_xyz}" rpy="${origin_rpy}"/>
       </collision>
-      <inertial>
-        <mass value="${mass}"/>
-        <origin xyz="${xyz}" rpy="${rpy}"/>
-        <inertia
-          ixx="${(1/12.0)*mass*(h*h + d*d)}"
-          iyy="${(1/12.0)*mass*(w*w + d*d)}"
-          izz="${(1/12.0)*mass*(w*w + h*h)}"
-          ixy="0.0" ixz="0.0" iyz="0.0"/>
-      </inertial>
     </link>
   </xacro:macro>
-  <!-- Macro for revolute or prismatic joint -->
-  <xacro:macro name="joint" params="name type parent child axis lower upper velocity effort xyz rpy">
+  <!-- ====== UNIFIED JOINT MACRO ====== -->
+  <xacro:macro name="cobot_joint" params="name type parent child axis limit_l limit_u limit_v limit_e origin_xyz origin_rpy">
     <joint name="${name}" type="${type}">
       <parent link="${parent}"/>
       <child link="${child}"/>
-      <axis xyz="${axis}"/>
-      <limit lower="${lower}" upper="${upper}" velocity="${velocity}" effort="${effort}"/>
-      <origin xyz="${xyz}" rpy="${rpy}"/>
+      <!-- Only add axis and limit for non-fixed joints -->
+      <xacro:if value="${type != 'fixed'}">
+        <axis xyz="${axis}"/>
+        <limit lower="${limit_l}" upper="${limit_u}" velocity="${limit_v}" effort="${limit_e}"/>
+      </xacro:if>
+      <origin xyz="${origin_xyz}" rpy="${origin_rpy}"/>
     </joint>
   </xacro:macro>
-  <!-- Macro for fixed joint -->
-  <xacro:macro name="fixed_joint" params="name parent child xyz rpy">
-    <joint name="${name}" type="fixed">
-      <parent link="${parent}"/>
-      <child link="${child}"/>
-      <origin xyz="${xyz}" rpy="${rpy}"/>
-    </joint>
-  </xacro:macro>
-  <!-- Macro for effort transmission -->
-  <!-- <xacro:macro name="transmission_effort" params="name joint_name actuator_name">
-    <transmission name="${name}">
-      <type>transmission_interface/SimpleTransmission</type>
-      <joint name="${joint_name}">
-        <hardwareInterface>hardware_interface/PositionJointInterface</hardwareInterface>
-      </joint>
-      <actuator name="${actuator_name}">
-        <hardwareInterface>hardware_interface/PositionJointInterface</hardwareInterface>
-        <mechanicalReduction>1</mechanicalReduction>
-      </actuator>
-    </transmission>
-  </xacro:macro> -->
 </robot>
