Commit message: stable vs unstable robots (without namespace vs applying namespace)

File: src/learn_robotics_with_ROS_youtube_channel/my_multi_robot/my_robot_description/urdf/my_robot.gazebo.xacro (robot description, xacro)
@@ -1,20 +1,30 @@
 <?xml version="1.0"?>
 <robot xmlns:xacro="http://www.ros.org/wiki/xacro">
-  <!-- ==================== GAZEBO ROS2 CONTROL PLUGIN ==================== -->
+  <!-- Multi-robot support: Get robot_name from parent -->
+  <xacro:arg name="robot_name" default="robot1"/>
+  <xacro:property name="robot_ns" value="$(arg robot_name)"/>
+  <!-- ==================== GAZEBO ROS 2 CONTROL PLUGIN ==================== -->
   <gazebo>
-    <plugin name="gz_ros2_control::GazeboSimROS2ControlPlugin" filename="libgz_ros2_control-system">
+    <plugin name="gz_ros2_control::GazeboSimROS2ControlPlugin"
+            filename="gz_ros2_control-system">
       <parameters>$(find my_robot_description)/config/robot_controller.yaml</parameters>
-      <controller_manager_name>controller_manager</controller_manager_name>
+      <ros>
+        <namespace>$(arg robot_name)</namespace>
+      </ros>
     </plugin>
   </gazebo>
-  <!-- ==================== LINK PHYSICS PROPERTIES ==================== -->
-  <!-- First Link Physics -->
-  <gazebo reference="first_link">
+  <!-- Make world link static in Gazebo -->
+  <gazebo reference="${robot_ns}/world">
+    <static>true</static>
+  </gazebo>
+  <!-- ==================== LINK GAZEBO PROPERTIES ==================== -->
+  <!-- First link: friction and visual material -->
+  <gazebo reference="${robot_ns}/first_link">
     <mu1>0.2</mu1>
     <mu2>0.2</mu2>
     <material>Gazebo/Red</material>
   </gazebo>
-  <!-- Second Link Physics -->
-  <gazebo reference="second_link">
+  <!-- Second link: friction and visual material -->
+  <gazebo reference="${robot_ns}/second_link">
     <mu1>0.2</mu1>
     <mu2>0.2</mu2>

File: src/learn_robotics_with_ROS_youtube_channel/my_multi_robot/my_robot_description/urdf/my_robot.urdf.xacro (robot description, xacro)
@@ -1,17 +1,15 @@
 <?xml version="1.0"?>
 <robot name="my_robot" xmlns:xacro="http://www.ros.org/wiki/xacro">
-  <!-- Include parameter definitions -->
-  <xacro:include filename="$(find my_robot_description)/urdf/parameters.xacro" />
-  <!-- Include Gazebo configuration -->
-  <xacro:include filename="$(find my_robot_description)/urdf/my_robot.gazebo.xacro" />
-  <!-- ==================== BASE LINK (World) ==================== -->
-  <link name="world"/>
-  <!-- ==================== FIXED JOINT ==================== -->
-  <joint name="world_to_first_link" type="fixed">
-    <parent link="world"/>
-    <child link="first_link"/>
-  </joint>
-  <!-- ==================== FIRST LINK ==================== -->
-  <link name="first_link">
+  <!-- Include external files -->
+  <xacro:include filename="$(find my_robot_description)/urdf/parameters.xacro"/>
+  <xacro:include filename="$(find my_robot_description)/urdf/my_robot.gazebo.xacro"/>
+  <!-- Multi-robot support: Accept robot_name as argument -->
+  <xacro:arg name="robot_name" default="robot1"/>
+  <xacro:property name="robot_ns" value="$(arg robot_name)"/>
+  <!-- ==================== LINKS ==================== -->
+  <!-- Base link (world frame) -->
+  <link name="${robot_ns}/world"/>
+  <!-- First link -->
+  <link name="${robot_ns}/first_link">
     <visual>
       <geometry>
@@ -29,15 +27,6 @@
     <xacro:inertial_section/>
   </link>
-  <!-- ==================== REVOLUTE JOINT ==================== -->
-  <joint name="first_joint" type="revolute">
-    <parent link="first_link"/>
-    <child link="second_link"/>
-    <origin xyz="0 ${b} ${q}" rpy="0 0 0"/>
-    <axis xyz="0 1 0"/>
-    <limit effort="${joint_effort}" velocity="${joint_velocity}" lower="${joint_lower}" upper="${joint_upper}"/>
-    <dynamics damping="${joint_damping}" friction="${joint_friction}"/>
-  </joint>
-  <!-- ==================== SECOND LINK ==================== -->
-  <link name="second_link">
+  <!-- Second link -->
+  <link name="${robot_ns}/second_link">
     <visual>
       <geometry>
@@ -55,13 +44,29 @@
     <xacro:inertial_section/>
   </link>
-  <!-- ==================== ROS2 CONTROL ==================== -->
+  <!-- ==================== JOINTS ==================== -->
+  <!-- Fixed joint: world to first link -->
+  <joint name="${robot_ns}/world_to_first_link" type="fixed">
+    <parent link="${robot_ns}/world"/>
+    <child link="${robot_ns}/first_link"/>
+  </joint>
+  <!-- Revolute joint: first link to second link -->
+    <joint name="${robot_ns}/first_joint" type="revolute">
+      <parent link="${robot_ns}/first_link"/>
+      <child link="${robot_ns}/second_link"/>
+      <origin xyz="0 ${b} ${q}" rpy="0 0 0"/>
+      <axis xyz="0 1 0"/>
+      <limit effort="${joint_effort}" velocity="${joint_velocity}"
+              lower="${joint_lower}" upper="${joint_upper}"/>
+      <dynamics damping="${joint_damping}" friction="${joint_friction}"/>
+    </joint>
+  <!-- ==================== ROS 2 CONTROL ==================== -->
   <ros2_control name="RobotController" type="system">
     <hardware>
       <plugin>gz_ros2_control/GazeboSimSystem</plugin>
     </hardware>
-    <joint name="first_joint">
+    <joint name="${robot_ns}/first_joint">
       <command_interface name="position">
-        <param name="min">${joint_lower}</param>
-        <param name="max">${joint_upper}</param>
+        <param name="min">-1.57</param>
+        <param name="max">1.57</param>
       </command_interface>
       <state_interface name="position"/>

File: src/learn_robotics_with_ROS_youtube_channel/my_multi_robot/my_robot_description/urdf/parameters.xacro (robot description, xacro)
@@ -2,25 +2,28 @@
 <robot xmlns:xacro="http://www.ros.org/wiki/xacro">
   <!-- ==================== GEOMETRIC PARAMETERS ==================== -->
-  <xacro:property name="a" value="0.1" />
-  <xacro:property name="b" value="0.1" />
-  <xacro:property name="c" value="0.8" />
+  <!-- Link dimensions (box geometry) -->
+  <xacro:property name="a" value="0.1"/>  <!-- Width (m) -->
+  <xacro:property name="b" value="0.1"/>  <!-- Depth (m) -->
+  <xacro:property name="c" value="0.8"/>  <!-- Height (m) -->
   <!-- ==================== CALCULATED PARAMETERS ==================== -->
-  <xacro:property name="s" value="${c/2}" />
-  <xacro:property name="q" value="${c-(c/4)}" />
+  <xacro:property name="s" value="${c/2}"/>        <!-- Half height for COM -->
+  <xacro:property name="q" value="${c-(c/4)}"/>    <!-- Joint offset from base -->
   <!-- ==================== MATERIAL PROPERTIES ==================== -->
-  <xacro:property name="d" value="2710" />
-  <xacro:property name="m" value="${d*a*b*c}" />
+  <xacro:property name="d" value="2710"/>          <!-- Density (kg/m³) - Aluminum -->
+  <xacro:property name="m" value="${d*a*b*c}"/>    <!-- Mass (kg) -->
   <!-- ==================== INERTIA CALCULATIONS ==================== -->
-  <xacro:property name="ix" value="${m*(b*b+c*c)/12}" />
-  <xacro:property name="iy" value="${m*(a*a+c*c)/12}" />
-  <xacro:property name="iz" value="${m*(a*a+b*b)/12}" />
+  <!-- Box inertia tensor (centered at origin) -->
+  <xacro:property name="ix" value="${m*(b*b+c*c)/12}"/>
+  <xacro:property name="iy" value="${m*(a*a+c*c)/12}"/>
+  <xacro:property name="iz" value="${m*(a*a+b*b)/12}"/>
   <!-- ==================== JOINT PARAMETERS ==================== -->
-  <xacro:property name="joint_effort" value="5000" />
-  <xacro:property name="joint_velocity" value="10" />
-  <xacro:property name="joint_lower" value="-1.57" />
-  <xacro:property name="joint_upper" value="1.57" />
-  <xacro:property name="joint_damping" value="1.0" />
-  <xacro:property name="joint_friction" value="1.0" />
+  <xacro:property name="joint_effort" value="5000"/>      <!-- Max torque (N·m) -->
+  <xacro:property name="joint_velocity" value="10"/>      <!-- Max velocity (rad/s) -->
+  <xacro:property name="joint_lower" value="-1.57"/>      <!-- Min angle (-90°) -->
+  <xacro:property name="joint_upper" value="1.57"/>       <!-- Max angle (+90°) -->
+  <xacro:property name="joint_damping" value="1.0"/>      <!-- Damping (N·m·s/rad) -->
+  <xacro:property name="joint_friction" value="1.0"/>     <!-- Static friction (N·m) -->
   <!-- ==================== INERTIAL MACRO ==================== -->
+  <!-- Reusable inertial properties for box links -->
   <xacro:macro name="inertial_section">
     <inertial>
@@ -33,9 +36,9 @@
   </xacro:macro>
   <!-- ==================== MATERIAL DEFINITIONS ==================== -->
+  <material name="red">
+    <color rgba="1 0 0 1"/>
+  </material>
   <material name="blue">
     <color rgba="0 0 1 1"/>
   </material>
-  <material name="red">
-    <color rgba="1 0 0 1"/>
-  </material>
 </robot>
